File: gateway/hw/ax-gateway.sch (KiCad schematic (older format))
At the start: 90 parts, among them IC1 TG-5006CJ, IC2 TPS73433, IC3 AX5243, IC4 AX5243, P1 Raspberry_Pi_Conn, P2 COAX, P3 COAX, P4 PAD

Commit message: [gateway] fix farnell code for shield
Parts:
- P4: Farnell 2497719 -> 2497723
Changed lines of the file:
@@
 F 2 "rem:BMI-S-x05" H 10400 5450 50  0001 L CNN
 F 3 "" H 10400 5600 50  0001 C CNN
-F 4 "2497719" H 10400 5600 60  0001 C CNN "Farnell"
+F 4 "2497723" H 10400 5600 60  0001 C CNN "Farnell"
 	1    10400 5600
 	0    -1   -1   0

Commit message: [hw] add l_ext
Parts:
- added L17, L18: 0Ω, agg:0402, symbol L_Small
Connections:
- net SYNTH_LOOP_0 renamed L1_0
- net L1_0: now also L17.1; no longer IC3.8 (L1)
- net SYNTH_LOOP_1 renamed L1_1
- net L1_1: now also L18.1; no longer IC4.8 (L1)
- new net L2_0: IC3.8 (L1), L17.2
- new net L2_1: IC4.8 (L1), L18.2
Other:
- note added: "Lext"

Commit message: [pi hw] add l_ext
Parts:
- L17, L18: value 0Ω -> 22nH; footprint agg:0402 -> agg:0603; STD.PAS 0Ω -> 22nH
Changed lines of the file:
@@
 EESchema Schematic File Version 2
-LIBS:power
+LIBS:ax5243
+LIBS:as213-92
+LIBS:bgm1034n7
+LIBS:bgu7003w
 LIBS:ax-gateway-cache
 EELAYER 25 0
@@
 Title "ax-gateway"
 Date "2016-06-04"
-Rev "v0.1"
+Rev "v0.4"
 Comp "Bristol SEDS"
 Comment1 "Richard Meadows"
@@
 P 5700 2800
 F 0 "L17" H 5550 2850 50  0000 L CNN
-F 1 "0Ω" H 5550 2750 50  0000 L CNN
-F 2 "agg:0402" H 5700 2800 50  0001 C CNN
+F 1 "22nH" H 5500 2750 50  0000 L CNN
+F 2 "agg:0603" H 5700 2800 50  0001 C CNN
 F 3 "" H 5700 2800 50  0000 C CNN
-F 4 "0Ω" H 5700 2800 60  0001 C CNN "STD.PAS"
+F 4 "22nH" H 5700 2800 60  0001 C CNN "STD.PAS"
 	1    5700 2800
 	-1   0    0    -1
@@
 P 5700 4900
 F 0 "L18" H 5550 4950 50  0000 L CNN
-F 1 "0Ω" H 5550 4850 50  0000 L CNN
-F 2 "agg:0402" H 5700 4900 50  0001 C CNN
+F 1 "22nH" H 5500 4850 50  0000 L CNN
+F 2 "agg:0603" H 5700 4900 50  0001 C CNN
 F 3 "" H 5700 4900 50  0000 C CNN
-F 4 "0Ω" H 5700 4900 60  0001 C CNN "STD.PAS"
+F 4 "22nH" H 5700 4900 60  0001 C CNN "STD.PAS"
 	1    5700 4900
 	-1   0    0    -1
