File: gateway/hw/panel/panel.kicad_pcb (KiCad board)
At the start: 2 copper layers, 100 x 80 mm, 132 parts, among them IC1 TG-5006CJ, IC2 TPS73433, IC3 AX5243, IC4 AX5243, P1 Raspberry_Pi_Conn, P2 COAX, P3 COAX, P4 PAD

Commit message: [pi hw] add l_ext
Parts:
- added L17: 22nH, agg:0603, F.Cu at (162.2, 104.0)
- added L18: 22nH, agg:0603, F.Cu at (162.8, 122.0)
- moved C1 4.04 mm to (167.0, 103.0), turned to 0 degrees
- moved P2 0.50 mm to (140.0, 100.0)
- moved P3 0.50 mm to (140.0, 118.0)
- moved C15 0.25 mm to (160.2, 103.8)
- moved C18 0.25 mm to (160.8, 121.8)
Connections:
- IC3 pad 7: /SYNTH_LOOP_0 -> /L1_0
- IC3 pad 8: /SYNTH_LOOP_0 -> /L2_0
- IC4 pad 7: /SYNTH_LOOP_1 -> /L1_1
- IC4 pad 8: /SYNTH_LOOP_1 -> /L2_1
Routing:
- net /L2_1: track 0.00 -> 2.82 mm
- net /L2_0: track 0.00 -> 2.82 mm
- net /L1_1: track 0.00 -> 2.34 mm
- net /L1_0: track 0.00 -> 2.34 mm
- net VDD: track 79.8 -> 78.8 mm
- net GND: track 476.0 -> 477.0 mm, vias 191 -> 192
- net /SYNTH_LOOP_1: track 0.50 -> 0.00 mm
- net /SYNTH_LOOP_0: track 0.50 -> 0.00 mm
- net (no net): vias 2 -> 0
Other:
- board text added: "Richard Meadows"
- board text added: "ax gateway v0.4 15-11-16"
- board text removed: "ax gateway v0.1 03-08-16 Richard Meadows"
